File: ergogen/kicad/production.kicad_pcb (KiCad board)
At the start: 2 copper layers, 143.3 x 107 mm, 41 parts

Commit message: Did wiring for 'v1.0.0'.
Parts:
- D1, D10, D11, D12, D13, D14, D15, D16, D17, D18, D19, D2, D3, D4, D5, D6, D7, D8, D9: moved to F.Cu
Routing:
- net (no net): track 262.1 -> 0.00 mm
- net P7: track 0.00 -> 212.3 mm, vias 1 -> 2
- net P6: track 0.00 -> 193.4 mm
- net P8: track 0.00 -> 184.3 mm, vias 1 -> 2
- net P9: track 0.00 -> 179.2 mm
- net P0: track 0.00 -> 161.3 mm
- net P4: track 0.00 -> 133.2 mm
- net P21: track 0.00 -> 130.4 mm
- net P1: track 0.00 -> 127.8 mm
- net P5: track 0.00 -> 108.4 mm
- net P20: track 0.00 -> 95.7 mm
- net VCC: track 0.00 -> 80.9 mm
- net GND: track 0.00 -> 78.6 mm
- net RST: track 0.00 -> 63.7 mm, vias 1 -> 3
- net P19: track 0.00 -> 62.8 mm
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Other:
- net class Default removed
- board text added: "Snowflake: v1.0.0"
- board text removed: "Version: v1.0.0"
